File: PCB/Sender/RcSender.kicad_pcb (KiCad board)
At the start: 2 copper layers, 90 x 60 mm, 48 parts, among them J1 USB_A, J2 Bat, J3 Prog, Q1 BC846BS, SW1 SW_Push, SW2 SW_Push, SW3 SW_Push, SW4 SW_Push, U1 MCP73832-2-OT, U2 AP2112K-3.3, U3 USBLC6-2SC6, U4 ESP32-WROOM-32, U5 COM-09032, U6 COM-09032, U7 CP2102N-Axx-xQFN28, U8 OLED128x64

Commit message: dual pwm fungere
Parts:
- moved R11 26.1 mm to (36.4, 88.7)
Connections:
- POT1 pad 2: IO5 -> IO36
- POT2 pad 2: IO4 -> IO39
- R11 pad 1: IO35 -> IO14
- U4 pad 4: unconnected-(U4-SENSOR_VP-Pad4) -> IO36
- U4 pad 5: unconnected-(U4-SENSOR_VN-Pad5) -> IO39
- U4 pad 6: /STDEsp32/GPIO34 -> IO34
- U4 pad 8: /STDEsp32/GPIO32 -> IO32
- U4 pad 9: /STDEsp32/GPIO33 -> IO33
- U5 pad B1A: IO35 -> IO14
- U5 pad H2: IO17 -> IO33
- U5 pad V2: IO18 -> IO32
- U6 pad H2: IO16 -> IO35
- U6 pad V2: IO14 -> IO34
Routing:
- net IO36: track 0.00 -> 68.3 mm
- net IO18: track 56.5 -> 1.77 mm
- net IO34: track 0.00 -> 54.6 mm, vias 0 -> 3
- net IO17: track 46.9 -> 2.13 mm
- net IO35: track 24.7 -> 66.0 mm, vias 1 -> 3
- net IO5: track 54.7 -> 13.4 mm
- net IO16: track 35.7 -> 0.00 mm
- net IO32: track 0.00 -> 35.5 mm
- net IO39: track 0.00 -> 32.9 mm, vias 0 -> 2
- net IO33: track 0.00 -> 31.6 mm
- net IO4: track 7.09 -> 0.00 mm
- net +3.3V: track 43.2 -> 37.3 mm, vias 17 -> 16
- net IO14: track 36.1 -> 33.0 mm, vias 0 -> 1
