File: PCB/Sender/RcSender.kicad_sch (KiCad schematic)
At the start: 31 parts, among them J1 USB_A, J2 Bat, SW1 SW_Push, SW2 SW_Push, SW3 SW_Push, SW4 SW_Push, U1 MCP73832-2-OT, U2 AP2112K-3.3, U3 USBLC6-2SC6, U8 OLED128x64

Commit message: dual pwm fungere
Connections:
- net IO4: no longer POT2.2
- net IO5: no longer POT1.2
- new net IO36: POT1.2
- new net IO39: POT2.2
- no-connect marks 8 -> 4
Other:
- sheet STDEsp32 ports: added GPIO36, GPIO39; removed none
Changed lines of the file:
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@@
 	)
 	(no_connect
-		(at 170.18 76.2)
-	)
-	(no_connect
-		(at 170.18 73.66)
-	)
-	(no_connect
-		(at 170.18 78.74)
-	)
-	(no_connect
 		(at 170.18 68.58)
 	)
@@
 	)
 	(no_connect
-		(at 170.18 63.5)
-	)
-	(no_connect
 		(at 170.18 66.04)
 	)
@@
 	(wire
 		(pts
+			(xy 147.32 62.23) (xy 148.59 62.23)
+		)
+		(stroke
+			(width 0)
+			(type default)
+		)
+	)
+	(wire
+		(pts
 			(xy 207.01 49.53) (xy 209.55 49.53)
 		)
@@
 	(wire
 		(pts
+			(xy 170.18 73.66) (xy 175.26 73.66)
+		)
+		(stroke
+			(width 0)
+			(type default)
+		)
+	)
+	(wire
+		(pts
 			(xy 24.13 106.68) (xy 24.13 107.95)
 		)
@@
 	(wire
 		(pts
+			(xy 170.18 78.74) (xy 175.26 78.74)
+		)
+		(stroke
+			(width 0)
+			(type default)
+		)
+	)
+	(wire
+		(pts
 			(xy 110.49 74.93) (xy 113.03 74.93)
 		)
@@
 	(wire
 		(pts
+			(xy 170.18 76.2) (xy 175.26 76.2)
+		)
+		(stroke
+			(width 0)
+			(type default)
+		)
+	)
+	(wire
+		(pts
 			(xy 252.73 36.83) (xy 257.81 36.83)
 		)
@@
 	(wire
 		(pts
+			(xy 147.32 64.77) (xy 148.59 64.77)
+		)
+		(stroke
+			(width 0)
+			(type default)
+		)
+	)
+	(wire
+		(pts
 			(xy 38.1 106.68) (xy 24.13 106.68)
 		)
@@
 		)
 	)
+	(global_label "IO34"
+		(shape input)
+		(at 175.26 78.74 0)
+		(fields_autoplaced yes)
+		(effects
+			(font
+				(size 1.27 1.27)
+			)
+			(justify left)
+		)
+		(property "Intersheetrefs" "${INTERSHEET_REFS}"
+			(at 182.5995 78.74 0)
+			(effects
+				(font
+					(size 1.27 1.27)
+				)
+				(justify left)
+				(hide yes)
+			)
+		)
+	)
 	(global_label "RX"
 		(shape input)
@@
 	(global_label "IO14"
 		(shape input)
+		(at 208.28 31.75 180)
+		(fields_autoplaced yes)
+		(effects
+			(font
+				(size 1.27 1.27)
+			)
+			(justify right)
+		)
+		(property "Intersheetrefs" "${INTERSHEET_REFS}"
+			(at 200.9405 31.75 0)
+			(effects
+				(font
+					(size 1.27 1.27)
+				)
+				(justify right)
+				(hide yes)
+			)
+		)
+	)
+	(global_label "IO35"
+		(shape input)
+		(at 207.01 52.07 180)
+		(fields_autoplaced yes)
+		(effects
+			(font
+				(size 1.27 1.27)
+			)
+			(justify right)
+		)
+		(property "Intersheetrefs" "${INTERSHEET_REFS}"
+			(at 199.6705 52.07 0)
+			(effects
+				(font
+					(size 1.27 1.27)
+				)
+				(justify right)
+				(hide yes)
+			)
+		)
+	)
+	(global_label "IO34"
+		(shape input)
 		(at 207.01 49.53 180)
 		(fields_autoplaced yes)
@@
 		)
 	)
-	(global_label "IO4"
+	(global_label "IO15"
 		(shape input)
-		(at 248.92 93.98 180)
+		(at 252.73 25.4 90)
 		(fields_autoplaced yes)
 		(effects
@@
 				(size 1.27 1.27)
 			)
-			(justify right)
+			(justify left)
 		)
 		(property "Intersheetrefs" "${INTERSHEET_REFS}"
-			(at 242.79 93.98 0)
+			(at 252.6506 18.6326 90)
 			(effects
 				(font
 					(size 1.27 1.27)
 				)
-				(justify right)
+				(justify left)
 				(hide yes)
 			)
 		)
 	)
-	(global_label "IO15"
+	(global_label "IO33"
 		(shape input)
-		(at 252.73 25.4 90)
+		(at 209.55 27.94 180)
 		(fields_autoplaced yes)
 		(effects
@@
 				(size 1.27 1.27)
 			)
-			(justify left)
+			(justify right)
 		)
 		(property "Intersheetrefs" "${INTERSHEET_REFS}"
-			(at 252.6506 18.6326 90)
+			(at 202.2105 27.94 0)
 			(effects
 				(font
 					(size 1.27 1.27)
 				)
-				(justify left)
+				(justify right)
 				(hide yes)
 			)
 		)
 	)
-	(global_label "IO17"
+	(global_label "BT"
 		(shape input)
-		(at 209.55 27.94 180)
+		(at 144.78 40.64 180)
 		(fields_autoplaced yes)
 		(effects
@@
 		)
 		(property "Intersheetrefs" "${INTERSHEET_REFS}"
-			(at 202.2105 27.94 0)
+			(at 139.5572 40.64 0)
 			(effects
 				(font
@@
 		)
 	)
-	(global_label "BT"
+	(global_label "IO34"
 		(shape input)
-		(at 144.78 40.64 180)
+		(at 187.96 20.32 180)
 		(fields_autoplaced yes)
 		(effects
@@
 		)
 		(property "Intersheetrefs" "${INTERSHEET_REFS}"
-			(at 139.5572 40.64 0)
+			(at 180.6205 20.32 0)
 			(effects
 				(font
@@
 	(global_label "IO35"
 		(shape input)
-		(at 208.28 31.75 180)
+		(at 195.58 29.21 180)
 		(fields_autoplaced yes)
 		(effects
@@
 		)
 		(property "Intersheetrefs" "${INTERSHEET_REFS}"
-			(at 200.9405 31.75 0)
+			(at 188.2405 29.21 0)
 			(effects
 				(font
@@
 		)
 	)
+	(global_label "IO32"
+		(shape input)
+		(at 175.26 73.66 0)
+		(fields_autoplaced yes)
+		(effects
+			(font
+				(size 1.27 1.27)
+			)
+			(justify left)
+		)
+		(property "Intersheetrefs" "${INTERSHEET_REFS}"
+			(at 182.5995 73.66 0)
+			(effects
+				(font
+					(size 1.27 1.27)
+				)
+				(justify left)
+				(hide yes)
+			)
+		)
+	)
 	(global_label "SCL"
 		(shape input)
@@
 		)
 	)
-	(global_label "IO18"
+	(global_label "IO39"
+		(shape input)
+		(at 147.32 64.77 180)
+		(fields_autoplaced yes)
+		(effects
+			(font
+				(size 1.27 1.27)
+			)
+			(justify right)
+		)
+		(property "Intersheetrefs" "${INTERSHEET_REFS}"
+			(at 139.9805 64.77 0)
+			(effects
+				(font
+					(size 1.27 1.27)
+				)
+				(justify right)
+				(hide yes)
+			)
+		)
+	)
+	(global_label "IO32"
 		(shape input)
 		(at 209.55 25.4 180)
@@
 		)
 	)
+	(global_label "IO39"
+		(shape input)
+		(at 248.92 93.98 180)
+		(fields_autoplaced yes)
+		(effects
+			(font
+				(size 1.27 1.27)
+			)
+			(justify right)
+		)
+		(property "Intersheetrefs" "${INTERSHEET_REFS}"
+			(at 241.5805 93.98 0)
+			(effects
+				(font
+					(size 1.27 1.27)
+				)
+				(justify right)
+				(hide yes)
+			)
+		)
+	)
 	(global_label "BT"
 		(shape input)
@@
 		)
 	)
-	(global_label "IO5"
+	(global_label "IO36"
+		(shape input)
+		(at 147.32 62.23 180)
+		(fields_autoplaced yes)
+		(effects
+			(font
+				(size 1.27 1.27)
+			)
+			(justify right)
+		)
+		(property "Intersheetrefs" "${INTERSHEET_REFS}"
+			(at 139.9805 62.23 0)
+			(effects
+				(font
+					(size 1.27 1.27)
+				)
+				(justify right)
+				(hide yes)
+			)
+		)
+	)
+	(global_label "IO36"
 		(shape input)
 		(at 248.92 77.47 180)
@@
 		)
 		(property "Intersheetrefs" "${INTERSHEET_REFS}"
-			(at 242.79 77.47 0)
+			(at 241.5805 77.47 0)
 			(effects
 				(font
@@
 		)
 	)
+	(global_label "IO33"
+		(shape input)
+		(at 175.26 76.2 0)
+		(fields_autoplaced yes)
+		(effects
+			(font
+				(size 1.27 1.27)
+			)
+			(justify left)
+		)
+		(property "Intersheetrefs" "${INTERSHEET_REFS}"
+			(at 182.5995 76.2 0)
+			(effects
+				(font
+					(size 1.27 1.27)
+				)
+				(justify left)
+				(hide yes)
+			)
+		)
+	)
 	(global_label "IO12"
 		(shape input)
@@
 		)
 	)
-	(global_label "IO16"
-		(shape input)
-		(at 207.01 52.07 180)
-		(fields_autoplaced yes)
-		(effects
-			(font
-				(size 1.27 1.27)
-			)
-			(justify right)
-		)
-		(property "Intersheetrefs" "${INTERSHEET_REFS}"
-			(at 199.6705 52.07 0)
-			(effects
-				(font
-					(size 1.27 1.27)
-				)
-				(justify right)
-				(hide yes)
-			)
-		)
-	)
 	(symbol
 		(lib_id "power:+3V3")
@@
 			)
 		)
+		(pin "GPIO36" input
+			(at 148.59 62.23 180)
+			(effects
+				(font
+					(size 1.27 1.27)
+				)
+				(justify left)
+			)
+		)
+		(pin "GPIO39" input
+			(at 148.59 64.77 180)
+			(effects
+				(font
+					(size 1.27 1.27)
+				)
+				(justify left)
+			)
+		)
