File: PCB/Sender/StdEsp32_worm2.kicad_sch (KiCad schematic)
At the start: 7 parts, among them J3 Prog, U4 ESP32-WROOM-32

Commit message: dual pwm fungere
Connections:
- net GPIO36: now reaches U4.4 (SENSOR_VP)
- net GPIO39: now reaches U4.5 (SENSOR_VN)
Other:
- moved on the sheet: C6, C7, C8, J3, R10, R9, U4
